Commit message: fork adding prototype of symulation in gazebo world.launch

File: magni_description/urdf/magni.urdf.xacro (robot description, xacro)
@@ -166,5 +166,5 @@
     <xacro:if value="${raspicam_mount == 'downward'}">
       <xacro:raspi_camera name="raspicam" connected_to="base_link">
-        <origin xyz="0.110 0.090 0.455" rpy="3.14159 -0.7854 0.0"/>
+        <origin xyz="0.110 0.090 0.255" rpy="3.14159 -0.7854 0.0"/>
       </xacro:raspi_camera>
     </xacro:if>

Commit message: added modified move_basic, fixed sonar cones, corrected camera resolution and position, changed sonar topics to reflect the real robot

File: magni_description/urdf/magni.urdf.xacro (robot description, xacro)
@@ -13,5 +13,5 @@
   <xacro:include filename="$(find magni_description)/urdf/inertial.xacro" />
   <xacro:include filename="$(find magni_description)/urdf/sensors/sonar_hc-sr04.xacro" />
-  <xacro:include filename="$(find magni_description)/urdf/sensors/raspi_camera.xacro" />
+  <xacro:include filename="$(find magni_description)/urdf/sensors/raspi_camera_v2.xacro" />
   <!-- Robot base_link -->
   <link name="base_link">
@@ -166,5 +166,5 @@
     <xacro:if value="${raspicam_mount == 'downward'}">
       <xacro:raspi_camera name="raspicam" connected_to="base_link">
-        <origin xyz="0.110 0.090 0.255" rpy="3.14159 -0.7854 0.0"/>
+        <origin xyz="0.1 0.090 0.145" rpy="3.14159 -1.25 0.0"/>
       </xacro:raspi_camera>
     </xacro:if>
